File: keyboard.kicad_pcb (KiCad board)
At the start: 2 copper layers, 344.2 x 121.9 mm, 137 parts, among them SW1 SW_Push, SW10 SW_Push, SW11 SW_Push, SW12 SW_Push, SW13 SW_Push, SW14 SW_Push, SW15 SW_Push, SW16 SW_Push, SW17 SW_Push, SW18 SW_Push, SW19 SW_Push, SW2 SW_Push, SW20 SW_Push, SW21 SW_Push, SW22 SW_Push, SW23 SW_Push, SW24 SW_Push, SW25 SW_Push, SW26 SW_Push, SW27 SW_Push, SW28 SW_Push, SW29 SW_Push, SW3 SW_Push, SW30 SW_Push, SW31 SW_Push, SW32 SW_Push, SW33 SW_Push, SW34 SW_Push, SW35 SW_Push, SW36 SW_Push, SW37 SW_Push, SW38 SW_Push, SW39 SW_Push, SW4 SW_Push, SW40 SW_Push, SW41 SW_Push, SW42 SW_Push, SW43 SW_Push, SW44 SW_Push, SW45 SW_Push, SW46 SW_Push, SW47 SW_Push, SW48 SW_Push, SW49 SW_Push, SW5 SW_Push, SW50 SW_Push, SW51 SW_Push, SW52 SW_Push, SW53 SW_Push, SW54 SW_Push, SW55 SW_Push, SW56 SW_Push, SW57 SW_Push, SW58 SW_Push, SW59 SW_Push, SW6 SW_Push, SW60 SW_Push, SW61 SW_Push, SW62 SW_Push, SW63 SW_Push, SW64 SW_Push, SW7 SW_Push, SW8 SW_Push, SW9 SW_Push, U1 Pro Micro, U2 TRRS, U3 Pro Micro, U4 TRRS

Commit message: Remove second connection from TRRS and ProMicro, redo traces on PCB to be cleaner
Parts:
- U1: moved to B.Cu
- moved U2 3.97 mm to (183.4, 154.0)
- moved U4 0.20 mm to (188.3, 154.0)
Connections:
- net SCL1 renamed TX1
- net SCL2 renamed TX2
- U1 pad 5: SDA1 -> unconnected-(U1-2/PD1-Pad5)
- U2 pad 4: SDA1 -> unconnected-(U2-RING2-Pad4)
- U3 pad 5: SDA2 -> unconnected-(U3-2/PD1-Pad5)
- U4 pad 4: SDA2 -> unconnected-(U4-RING2-Pad4)
Routing:
- net VCC: track 388.2 -> 0.00 mm, vias 8 -> 0
- net SDA1: track 253.9 -> 0.00 mm, vias 3 -> 0
- net TX1: track 238.7 -> 0.00 mm, vias 3 -> 0
- net SDA2: track 203.9 -> 0.00 mm, vias 4 -> 0
- net TX2: track 201.2 -> 0.00 mm, vias 4 -> 0
- net GND: track 394.5 -> 211.2 mm, vias 5 -> 0
- net COL9: track 208.7 -> 62.3 mm, vias 7 -> 6
- net COL6: track 269.5 -> 213.8 mm, vias 12 -> 10
- net COL10: track 211.2 -> 181.8 mm, vias 9 -> 10
- net ROW0: track 157.3 -> 134.2 mm, vias 1 -> 2
- net COL12: track 143.5 -> 122.0 mm, vias 7 -> 6
- net COL11: track 160.9 -> 142.8 mm
- net COL2: track 128.3 -> 111.8 mm, vias 9 -> 6
- net ROW3: track 183.1 -> 168.4 mm, vias 1 -> 2
- net ROW1: track 143.1 -> 128.9 mm, vias 1 -> 2
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
Commit message: Redo edge cuts, panelize PCB edge cuts
Parts:
- added REF**: breakaway-mousebites, random-keyboard-parts:breakaway-mousebites, F.Cu at (350.3, 81.5)
- added REF**: breakaway-mousebites, random-keyboard-parts:breakaway-mousebites, F.Cu at (305.1, 81.1)
- added REF**: breakaway-mousebites, random-keyboard-parts:breakaway-mousebites, F.Cu at (374.4, 184.2)
- added REF**: breakaway-mousebites, random-keyboard-parts:breakaway-mousebites, F.Cu at (90.9, 183.6)
- added REF**: breakaway-mousebites, random-keyboard-parts:breakaway-mousebites, F.Cu at (77.5, 81.2)
- added REF**: breakaway-mousebites, random-keyboard-parts:breakaway-mousebites, F.Cu at (115.3, 81.3)
- added REF**: breakaway-mousebites, random-keyboard-parts:breakaway-mousebites, F.Cu at (317.8, 184.2)
- added REF**: breakaway-mousebites, random-keyboard-parts:breakaway-mousebites, F.Cu at (54.6, 183.6)
- moved D10 19.5 mm to (123.8, 117.8)
- moved D13 19.5 mm to (179.7, 129.7)
- moved D14 19.5 mm to (78.5, 136.1)
- moved D18 19.5 mm to (161.8, 145.4)
- moved D19 19.5 mm to (180.4, 149.3)
- moved D2 19.5 mm to (98.0, 98.0)
- moved D20 19.5 mm to (79.4, 155.2)
- moved D21 19.5 mm to (110.4, 155.2)
- moved D22 19.5 mm to (129.9, 158.1)
- moved D23 19.5 mm to (148.5, 162.0)
- moved D24 19.5 mm to (167.2, 166.0)
- moved D25 19.5 mm to (185.8, 169.9)
- moved D26 19.5 mm to (76.1, 174.2)
- moved D27 19.5 mm to (99.9, 174.2)
- moved D3 19.5 mm to (117.0, 96.1)
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Routing:
- net VCC: track 0.00 -> 393.9 mm, vias 0 -> 7
- net TX2: track 0.00 -> 223.3 mm, vias 0 -> 2
- net GND: track 211.2 -> 399.5 mm, vias 0 -> 3
- net TX1: track 0.00 -> 176.6 mm, vias 0 -> 1
- net COL9: track 62.3 -> 93.7 mm
- net Net-(D34-A): track 0.00 -> 7.99 mm
- net COL10: track 181.8 -> 183.3 mm
- net COL2: track 111.8 -> 111.6 mm, vias 6 -> 7
Other:
- board size 344.2 x 121.9 mm -> 353.6 x 152.4 mm
- board text added: "TeaQueen by gregandcin"

Commit message: Add missing route
Routing:
- net COL9: track 93.7 -> 184.9 mm, vias 6 -> 9
- net COL11: track 142.8 -> 143.5 mm
Changed lines of the file:
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@@
   (segment (start 230.591142 123.025578) (end 231.616449 127.892898) (width 0.2) (layer "B.Cu") (net 93))
   (segment (start 365.760199 99.317898) (end 368.976356 99.037112) (width 0.2) (layer "B.Cu") (net 93))
+  (segment (start 318.522807 105.797807) (end 316.70625 103.98125) (width 0.2) (layer "F.Cu") (net 94))
   (segment (start 253.841449 102.492898) (end 253.841449 108.783551) (width 0.2) (layer "F.Cu") (net 94))
+  (segment (start 297.65625 99.21875) (end 295.275 101.6) (width 0.2) (layer "F.Cu") (net 94))
+  (segment (start 295.275 101.6) (end 293.6875 101.6) (width 0.2) (layer "F.Cu") (net 94))
   (segment (start 256.222699 142.180398) (end 254.635199 150.117898) (width 0.2) (layer "F.Cu") (net 94))
   (segment (start 253.841449 108.783551) (end 253.825 108.8) (width 0.2) (layer "F.Cu") (net 94))
   (segment (start 251.460199 123.924148) (end 254.635199 129.480398) (width 0.2) (layer "F.Cu") (net 94))
+  (segment (start 368.976356 101.577112) (end 364.755661 105.797807) (width 0.2) (layer "F.Cu") (net 94))
+  (segment (start 364.755661 105.797807) (end 318.522807 105.797807) (width 0.2) (layer "F.Cu") (net 94))
   (via (at 256.222699 142.180398) (size 0.6) (drill 0.3) (layers "F.Cu" "B.Cu") (net 94))
+  (via (at 293.6875 101.6) (size 0.6) (drill 0.3) (layers "F.Cu" "B.Cu") (net 94))
+  (via (at 316.70625 103.98125) (size 0.6) (drill 0.3) (layers "F.Cu" "B.Cu") (net 94))
   (via (at 253.841449 102.492898) (size 0.6) (drill 0.3) (layers "F.Cu" "B.Cu") (net 94))
+  (via (at 297.65625 99.21875) (size 0.6) (drill 0.3) (layers "F.Cu" "B.Cu") (net 94))
   (via (at 253.825 108.8) (size 0.6) (drill 0.3) (layers "F.Cu" "B.Cu") (net 94))
   (via (at 251.460199 123.924148) (size 0.6) (drill 0.3) (layers "F.Cu" "B.Cu") (net 94))
@@
   (via (at 254.635199 150.117898) (size 0.6) (drill 0.3) (layers "F.Cu" "B.Cu") (net 94))
   (segment (start 249.224854 113.400146) (end 249.224854 119.06486) (width 0.2) (layer "B.Cu") (net 94))
+  (segment (start 288.13125 101.6) (end 283.325 102.575) (width 0.2) (layer "B.Cu") (net 94))
   (segment (start 254.580992 98.450789) (end 253.841449 102.492898) (width 0.2) (layer "B.Cu") (net 94))
   (segment (start 254.635199 129.480398) (end 257.844 136.708392) (width 0.2) (layer "B.Cu") (net 94))
   (segment (start 253.825 108.8) (end 249.224854 113.400146) (width 0.2) (layer "B.Cu") (net 94))
+  (segment (start 311.94375 99.21875) (end 297.65625 99.21875) (width 0.2) (layer "B.Cu") (net 94))
   (segment (start 257.844 136.708392) (end 256.222699 142.180398) (width 0.2) (layer "B.Cu") (net 94))
+  (segment (start 316.70625 103.98125) (end 311.94375 99.21875) (width 0.2) (layer "B.Cu") (net 94))
+  (segment (start 293.6875 101.6) (end 288.13125 101.6) (width 0.2) (layer "B.Cu") (net 94))
   (segment (start 249.224854 119.06486) (end 251.460199 123.924148) (width 0.2) (layer "B.Cu") (net 94))
   (segment (start 253.825 108.8) (end 283.325 102.575) (width 0.2) (layer "B.Cu") (net 94))
   (segment (start 254.635199 150.117898) (end 252.487862 157.322463) (width 0.2) (layer "B.Cu") (net 94))
+  (segment (start 366.895661 106.197807) (end 317.247807 106.197807) (width 0.2) (layer "F.Cu") (net 95))
   (segment (start 287.178949 100.111648) (end 272.097699 100.111648) (width 0.2) (layer "F.Cu") (net 95))
   (segment (start 271.303949 157.261648) (end 274.478949 166.786648) (width 0.2) (layer "F.Cu") (net 95))
+  (segment (start 368.976356 104.117112) (end 366.895661 106.197807) (width 0.2) (layer "F.Cu") (net 95))
   (segment (start 272.097699 100.111648) (end 268.922699 108.049148) (width 0.2) (layer "F.Cu") (net 95))
   (segment (start 276.066449 137.417898) (end 273.685199 146.149148) (width 0.2) (layer "F.Cu") (net 95))
-  (segment (start 367.118468 105.975) (end 336.325 105.975) (width 0.2) (layer "F.Cu") (net 95))
+  (segment (start 317.247807 106.197807) (end 316.175 105.125) (width 0.2) (layer "F.Cu") (net 95))
   (segment (start 268.128949 119.161648) (end 273.685199 126.305398) (width 0.2) (layer "F.Cu") (net 95))
-  (segment (start 336.325 105.975) (end 317.025 105.975) (width 0.2) (layer "F.Cu") (net 95))
-  (segment (start 368.976356 104.117112) (end 367.118468 105.975) (width 0.2) (layer "F.Cu") (net 95))
-  (segment (start 317.025 105.975) (end 316.175 105.125) (width 0.2) (layer "F.Cu") (net 95))
   (via (at 276.066449 137.417898) (size 0.6) (drill 0.3) (layers "F.Cu" "B.Cu") (net 95))
   (via (at 273.685199 146.149148) (size 0.6) (drill 0.3) (layers "F.Cu" "B.Cu") (net 95))
@@
   (segment (start 316.175 105.125) (end 311.161648 100.111648) (width 0.2) (layer "B.Cu") (net 95))
   (segment (start 273.685199 126.305398) (end 276.477712 132.747675) (width 0.2) (layer "B.Cu") (net 95))
-  (segment (start 368.917051 106.597807) (end 315.890108 106.597807) (width 0.2) (layer "F.Cu") (net 96))
+  (segment (start 368.100056 107.533412) (end 362.783291 107.533412) (width 0.2) (layer "F.Cu") (net 96))
   (segment (start 288.766449 115.192898) (end 294.322699 123.130398) (width 0.2) (layer "F.Cu") (net 96))
+  (segment (start 362.783291 107.533412) (end 361.847686 106.597807) (width 0.2) (layer "F.Cu") (net 96))
   (segment (start 315.890108 106.597807) (end 314.960199 105.667898) (width 0.2) (layer "F.Cu") (net 96))
+  (segment (start 368.976356 106.657112) (end 368.100056 107.533412) (width 0.2) (layer "F.Cu") (net 96))
   (segment (start 292.735199 96.142898) (end 291.147699 102.492898) (width 0.2) (layer "F.Cu") (net 96))
+  (segment (start 361.847686 106.597807) (end 315.890108 106.597807) (width 0.2) (layer "F.Cu") (net 96))
   (segment (start 295.910199 135.036648) (end 294.322699 142.974148) (width 0.2) (layer "F.Cu") (net 96))
-  (segment (start 368.976356 106.657112) (end 368.917051 106.597807) (width 0.2) (layer "F.Cu") (net 96))
   (via (at 291.147699 102.492898) (size 0.6) (drill 0.3) (layers "F.Cu" "B.Cu") (net 96))
   (via (at 294.322699 123.130398) (size 0.6) (drill 0.3) (layers "F.Cu" "B.Cu") (net 96))
@@
   (segment (start 291.147699 102.492898) (end 288.972939 110.460307) (width 0.2) (layer "B.Cu") (net 96))
   (segment (start 294.322699 123.130398) (end 297.926439 130.462807) (width 0.2) (layer "B.Cu") (net 96))
-  (segment (start 366.777051 106.997807) (end 312.321358 106.997807) (width 0.2) (layer "F.Cu") (net 97))
   (segment (start 312.578949 96.142898) (end 310.197699 104.874148) (width 0.2) (layer "F.Cu") (net 97))
+  (segment (start 368.976356 109.197112) (end 363.881307 109.197112) (width 0.2) (layer "F.Cu") (net 97))
   (segment (start 307.816449 115.192898) (end 313.372699 123.924148) (width 0.2) (layer "F.Cu") (net 97))
+  (segment (start 363.881307 109.197112) (end 361.682002 106.997807) (width 0.2) (layer "F.Cu") (net 97))
+  (segment (start 361.682002 106.997807) (end 312.321358 106.997807) (width 0.2) (layer "F.Cu") (net 97))
   (segment (start 312.321358 106.997807) (end 310.197699 104.874148) (width 0.2) (layer "F.Cu") (net 97))
   (segment (start 314.960199 135.830398) (end 311.785199 142.974148) (width 0.2) (layer "F.Cu") (net 97))
-  (segment (start 368.976356 109.197112) (end 366.777051 106.997807) (width 0.2) (layer "F.Cu") (net 97))
   (via (at 314.960199 135.830398) (size 0.6) (drill 0.3) (layers "F.Cu" "B.Cu") (net 97))
   (via (at 313.372699 123.924148) (size 0.6) (drill 0.3) (layers "F.Cu" "B.Cu") (net 97))

Commit message: Redo some of the panels
Other:
- board size 353.6 x 152.4 mm -> 355 x 150.1 mm
Changed lines of the file:
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@@
   (gr_line (start 210.016849 203.376247) (end 299.676849 184.386247)
-    (stroke (width 0.05) (type default)) (layer "Edge.Cuts"))
-  (gr_line (start 377.075 208.325) (end 390.925 208.3)
     (stroke (width 0.05) (type default)) (layer "Edge.Cuts"))
   (gr_line (start 377.1 184.35) (end 385.703949 184.343949)
     (stroke (width 0.05) (type default)) (layer "Edge.Cuts"))
   (gr_line (start 74.85 81.025) (end 74.85 76.195)
-    (stroke (width 0.05) (type default)) (layer "Edge.Cuts"))
-  (gr_line (start 315 208.275) (end 314.756 208.275)
     (stroke (width 0.05) (type default)) (layer "Edge.Cuts"))
   (gr_line (start 353.05 81.35) (end 385.728949 81.563949)
@@
   (gr_line (start 320.85 208.275) (end 371.675 208.325)
     (stroke (width 0.05) (type default)) (layer "Edge.Cuts"))
+  (gr_line (start 36.5 217.275) (end 36.5 207.275)
+    (stroke (width 0.05) (type default)) (layer "Edge.Cuts"))
+  (gr_line (start 36.5 67.175) (end 36.5 76.2)
+    (stroke (width 0.05) (type default)) (layer "Edge.Cuts"))
+  (gr_line (start 391.5 67.175) (end 391.5 76.225)
+    (stroke (width 0.05) (type default)) (layer "Edge.Cuts"))
   (gr_line (start 93.65 183.825) (end 106.145319 183.826602)
     (stroke (width 0.05) (type default)) (layer "Edge.Cuts"))
@@
   (gr_line (start 118.1 76.2) (end 302.425 76.2)
     (stroke (width 0.05) (type default)) (layer "Edge.Cuts"))
-  (gr_line (start 390.918281 218.442563) (end 390.925 208.3)
-    (stroke (width 0.05) (type default)) (layer "Edge.Cuts"))
-  (gr_line (start 391 76.25) (end 391 66.25)
-    (stroke (width 0.05) (type default)) (layer "Edge.Cuts"))
   (gr_line (start 377.1 184.35) (end 377.075 208.325)
-    (stroke (width 0.05) (type default)) (layer "Edge.Cuts"))
-  (gr_line (start 38.7 217.475) (end 38.706719 207.332437)
     (stroke (width 0.05) (type default)) (layer "Edge.Cuts"))
   (gr_line (start 195.805319 202.816602) (end 199.635319 203.636601)
     (stroke (width 0.05) (type default)) (layer "Edge.Cuts"))
   (gr_line (start 80.125 76.195) (end 112.65 76.2)
-    (stroke (width 0.05) (type default)) (layer "Edge.Cuts"))
-  (gr_line (start 93.656719 207.334681) (end 314.756 208.275)
     (stroke (width 0.05) (type default)) (layer "Edge.Cuts"))
   (gr_line (start 57.35 183.825256) (end 57.356719 207.334937)
@@
   (gr_arc (start 385.728949 81.563949) (mid 387.525 82.307898) (end 388.268949 84.103949)
     (stroke (width 0.05) (type default)) (layer "Edge.Cuts"))
+  (gr_line (start 391.5 67.175) (end 36.5 67.175)
+    (stroke (width 0.05) (type default)) (layer "Edge.Cuts"))
   (gr_line (start 207.31185 99.516248) (end 207.286849 153.076248)
     (stroke (width 0.05) (type default)) (layer "Edge.Cuts"))
@@
   (gr_line (start 320.475 184.3) (end 320.475 208.275)
     (stroke (width 0.05) (type default)) (layer "Edge.Cuts"))
-  (gr_line (start 390.918281 218.442563) (end 38.7 217.475)
-    (stroke (width 0.05) (type default)) (layer "Edge.Cuts"))
   (gr_line (start 299.676849 184.386247) (end 313.738 184.38242)
     (stroke (width 0.05) (type default)) (layer "Edge.Cuts"))
@@
   (gr_line (start 112.65 81.06958) (end 112.65 76.2)
     (stroke (width 0.05) (type default)) (layer "Edge.Cuts"))
-  (gr_line (start 93.65 183.825) (end 93.656719 207.334681)
+  (gr_line (start 93.65 183.825) (end 93.656719 207.475)
     (stroke (width 0.05) (type default)) (layer "Edge.Cuts"))
   (gr_line (start 88.175 183.83242) (end 88.177 207.28742)
@@
   (gr_line (start 371.675 208.325) (end 371.677 207.28742)
     (stroke (width 0.05) (type default)) (layer "Edge.Cuts"))
-  (gr_line (start 391 66.25) (end 37.4 66.075)
-    (stroke (width 0.05) (type default)) (layer "Edge.Cuts"))
   (gr_line (start 42.345319 92.376602) (end 42.370319 181.286602)
     (stroke (width 0.05) (type default)) (layer "Edge.Cuts"))
   (gr_line (start 42.345319 92.376602) (end 42.345319 83.586602)
     (stroke (width 0.05) (type default)) (layer "Edge.Cuts"))
-  (gr_line (start 37.45 76.2) (end 37.4 66.075)
+  (gr_arc (start 207.314675 99.51625) (mid 207.785451 98.047595) (end 209.020823 97.124322)
     (stroke (width 0.05) (type default)) (layer "Edge.Cuts"))
-  (gr_arc (start 207.311851 99.516248) (mid 207.783151 98.045956) (end 209.0199 97.121653)
-    (stroke (width 0.05) (type default)) (layer "Edge.Cuts"))
-  (gr_line (start 353.05 76.225) (end 391 76.25)
+  (gr_line (start 51.877 207.28742) (end 36.5 207.275)
     (stroke (width 0.05) (type default)) (layer "Edge.Cuts"))
   (gr_line (start 353.05 81.35) (end 353.05 76.225)
@@
   (gr_line (start 74.85 81.025) (end 54.995319 81.046602)
     (stroke (width 0.05) (type default)) (layer "Edge.Cuts"))
+  (gr_line (start 315 208.275) (end 93.656719 207.475)
+    (stroke (width 0.05) (type default)) (layer "Edge.Cuts"))
+  (gr_line (start 74.85 76.195) (end 36.5 76.2)
+    (stroke (width 0.05) (type default)) (layer "Edge.Cuts"))
+  (gr_line (start 391.5 217.275) (end 391.5 208.25)
+    (stroke (width 0.05) (type default)) (layer "Edge.Cuts"))
   (gr_line (start 388.243949 181.803949) (end 388.268949 92.893949)
     (stroke (width 0.05) (type default)) (layer "Edge.Cuts"))
-  (gr_line (start 51.877 207.28742) (end 38.706719 207.332437)
+  (gr_line (start 36.5 217.275) (end 391.5 217.275)
     (stroke (width 0.05) (type default)) (layer "Edge.Cuts"))
   (gr_line (start 388.268949 84.103949) (end 388.268949 92.893949)
@@
   (gr_arc (start 42.344811 83.586602) (mid 43.071317 81.807962) (end 44.835319 81.046603)
     (stroke (width 0.05) (type default)) (layer "Edge.Cuts"))
+  (gr_line (start 377.075 208.325) (end 391.5 208.25)
+    (stroke (width 0.05) (type default)) (layer "Edge.Cuts"))
   (gr_line (start 202.365319 153.336602) (end 202.340318 99.776602)
-    (stroke (width 0.05) (type default)) (layer "Edge.Cuts"))
-  (gr_line (start 74.85 76.195) (end 37.45 76.2)
     (stroke (width 0.05) (type default)) (layer "Edge.Cuts"))
   (gr_line (start 118.1 81.075) (end 118.1 76.2)
     (stroke (width 0.05) (type default)) (layer "Edge.Cuts"))
+  (gr_line (start 353.05 76.225) (end 391.5 76.225)
+    (stroke (width 0.05) (type default)) (layer "Edge.Cuts"))
   (gr_text "TeaQueen\nby gregandcin" (at 312.75 171.825) (layer "F.SilkS")

Commit message: Redo reouting to reduce number of vias
Parts:
- moved ST37 0.45 mm to (348.8, 94.5)
Routing:
- net COL6: track 213.8 -> 242.0 mm, vias 10 -> 7
- net COL13: track 123.8 -> 148.1 mm, vias 6 -> 5
- net COL11: track 143.5 -> 165.0 mm, vias 7 -> 4
- net VCC: track 393.9 -> 415.2 mm, vias 7 -> 5
- net COL3: track 156.2 -> 176.7 mm, vias 9 -> 7
- net GND: track 399.5 -> 419.3 mm, vias 3 -> 4
- net COL10: track 183.5 -> 203.1 mm, vias 10 -> 6
- net COL5: track 192.3 -> 211.3 mm, vias 11 -> 7
- net COL12: track 122.0 -> 140.3 mm, vias 6 -> 4
- net COL8: track 234.5 -> 252.7 mm, vias 8 -> 6
- net ROW7: track 164.4 -> 181.8 mm, vias 0 -> 1
- net COL2: track 111.6 -> 128.0 mm, vias 7 -> 5
- net ROW9: track 185.4 -> 200.0 mm, vias 0 -> 1
- net COL14: track 88.3 -> 102.1 mm, vias 6 -> 4
- net COL7: track 234.6 -> 247.2 mm, vias 0 -> 6
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