File: keyboard.kicad_pcb (KiCad board)
At the start: 2 copper layers, 355 x 150.1 mm, 145 parts, among them SW1 SW_Push, SW10 SW_Push, SW11 SW_Push, SW12 SW_Push, SW13 SW_Push, SW14 SW_Push, SW15 SW_Push, SW16 SW_Push, SW17 SW_Push, SW18 SW_Push, SW19 SW_Push, SW2 SW_Push, SW20 SW_Push, SW21 SW_Push, SW22 SW_Push, SW23 SW_Push, SW24 SW_Push, SW25 SW_Push, SW26 SW_Push, SW27 SW_Push, SW28 SW_Push, SW29 SW_Push, SW3 SW_Push, SW30 SW_Push, SW31 SW_Push, SW32 SW_Push, SW33 SW_Push, SW34 SW_Push, SW35 SW_Push, SW36 SW_Push, SW37 SW_Push, SW38 SW_Push, SW39 SW_Push, SW4 SW_Push, SW40 SW_Push, SW41 SW_Push, SW42 SW_Push, SW43 SW_Push, SW44 SW_Push, SW45 SW_Push, SW46 SW_Push, SW47 SW_Push, SW48 SW_Push, SW49 SW_Push, SW5 SW_Push, SW50 SW_Push, SW51 SW_Push, SW52 SW_Push, SW53 SW_Push, SW54 SW_Push, SW55 SW_Push, SW56 SW_Push, SW57 SW_Push, SW58 SW_Push, SW59 SW_Push, SW6 SW_Push, SW60 SW_Push, SW61 SW_Push, SW62 SW_Push, SW63 SW_Push, SW64 SW_Push, SW7 SW_Push, SW8 SW_Push, SW9 SW_Push, U1 Pro Micro, U2 TRRS, U3 Pro Micro, U4 TRRS

Commit message: Update Diode names
Parts:
- D1, D10, D11, D12, D13, D14, D15, D16, D17, D18, D19, D2, D20, D21, D22, D23, D24, D25, D26, D27, D28, D29, D3, D30, D31, D32, D33, D34, D35, D36, D37, D38, D39, D4, D40, D41, D42, D43, D44, D45, D46, D47, D48, D49, D5, D50, D51, D52, D53, D54, D55, D56, D57, D58, D59, D6, D60, D61, D62, D63, D64, D7, D8, D9: value SOD_123 -> SOD_323F

Commit message: Change from SOD_323F to SOD_123 footprint for diodes
Parts:
- D1, D10, D11, D12, D13, D14, D15, D16, D17, D18, D19, D2, D20, D21, D22, D23, D24, D25, D26, D27, D28, D29, D3, D30, D31, D32, D33, D34, D35, D36, D37, D38, D39, D4, D40, D41, D42, D43, D44, D45, D46, D47, D48, D49, D5, D50, D51, D52, D53, D54, D55, D56, D57, D58, D59, D6, D60, D61, D62, D63, D64, D7, D8, D9: value SOD_323F -> SOD_123; footprint Diode_SMD:D_SOD-323F -> Diode_SMD:D_SOD-123
- moved D35 1.00 mm to (306.3, 97.0)
- moved D31 1.00 mm to (230.4, 110.3)
- moved D32 1.00 mm to (249.0, 106.3)
- moved D33 1.00 mm to (267.6, 102.4)
- moved D34 1.00 mm to (286.3, 98.4)
- moved D36 1.00 mm to (325.3, 98.9)
- moved D37 1.00 mm to (353.9, 98.9)
- moved D20 0.76 mm to (79.4, 155.9)
- moved D21 0.76 mm to (110.4, 155.9)
- moved D22 0.76 mm to (129.9, 158.8)
- moved D24 0.76 mm to (167.2, 166.7)
- moved D26 0.76 mm to (76.1, 175.0)
- moved D27 0.76 mm to (99.9, 175.0)
- moved D29 0.76 mm to (163.2, 185.4)
- moved D23 0.76 mm to (148.5, 162.8)
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Routing:
- net VCC: track 415.2 -> 411.3 mm
- net COL9: track 194.2 -> 197.6 mm
- net TX2: track 216.6 -> 218.5 mm
- net ROW5: track 162.0 -> 163.7 mm
- net COL6: track 241.7 -> 240.1 mm
- net ROW6: track 172.9 -> 174.1 mm
- net ROW9: track 200.0 -> 201.1 mm
- net ROW1: track 132.7 -> 133.6 mm
- net ROW7: track 181.8 -> 182.4 mm
- net ROW3: track 173.5 -> 174.1 mm
- net ROW4: track 202.3 -> 202.8 mm
- net ROW2: track 150.8 -> 151.3 mm
